File: Charger_MPPT/POWER.kicad_sch (KiCad schematic)
At the start: 48 parts, among them Q16 DMP3028LFD, Q6 BC847, U28 MC34063AD, U29 AP62200, U9 LM2596S-5

Commit message: added order link
Parts:
- C112: value 100uF/25V -> 100uF/16V; footprint Capacitor_Tantalum_SMD:CP_EIA-7343-43_Kemet-X -> Capacitor_Tantalum_SMD:CP_EIA-6032-20_AVX-F_Pad2.25x2.35mm_HandSolder; Order (none) -> https://lcsc.com/product-detail/Tantalum-Capacitors_Kyocera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
- C115: value 330uF/35V -> 100uF/16V; footprint Capacitor_Tantalum_SMD:CP_EIA-3216-10_Kemet-I -> Capacitor_Tantalum_SMD:CP_EIA-6032-15_Kemet-U; Order (none) -> https://lcsc.com/product-detail/Tantalum-Capacitors_Kyocera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
- C31: Order (none) -> https://lcsc.com/product-detail/image/CY2103MD1IEF4CC2A8_C2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
- C32, C34: value 330uF/16V -> 100uF/16V; Order (none) -> https://lcsc.com/product-detail/Tantalum-Capacitors_Kyocera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
- C33: Order (none) -> https://lcsc.com/product-detail/Tantalum-Capacitors_Kyocera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
- D51: Order (none) -> https://lcsc.com/product-detail/Schottky-Diodes_Guangdong-H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
- L6, L7: Order https://www.mouser.vn/ProductDetail/Pulse-Electronics/PA432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 -> https://lcsc.com/product-detail/image/CYA0650-33UH_C5189937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
- U28: Order https://www.mouser.vn/ProductDetail/Texas-Instruments/MC340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 -> https://lcsc.com/product-detail/image/MC34063ADR_C100023.ht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
- U9: Order https://www.thegioiic.com/lm2596s-5-0-ic-dieu-chinh-giam-ap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 -> https://lcsc.com/product-detail/image/LM2596S-5-0_C5276750.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
Changed lines of the file:
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@@
 			)
 		)
-		(property "Order" "https://www.thegioiic.com/lm2596s-5-0-ic-dieu-chinh-giam-ap-5v-3a-to-263-5"
+		(property "Order" "https://lcsc.com/product-detail/image/LM2596S-5-0_C5276750.html"
 			(at 190.5 140.97 0)
 			(effects
@@
 			)
 		)
+		(property "Order" "https://lcsc.com/product-detail/Schottky-Diodes_Guangdong-Hottech-1N5819WS_C191023.html?s_z=n_1n5819"
+			(at 223.52 109.22 0)
+			(effects
+				(font
+					(size 1.27 1.27)
+				)
+				(hide yes)
+			)
+		)
 		(pin "1"
 		)
@@
 			)
 		)
-		(property "Value" "100uF/25V"
+		(property "Value" "100uF/16V"
 			(at 234.95 109.22 0)
 			(effects
@@
 			)
 		)
-		(property "Footprint" "Capacitor_Tantalum_SMD:CP_EIA-7343-43_Kemet-X"
+		(property "Footprint" "Capacitor_Tantalum_SMD:CP_EIA-6032-20_AVX-F_Pad2.25x2.35mm_HandSolder"
 			(at 233.68 105.41 0)
 			(effects
@@
 			)
 		)
+		(property "Order" "https://lcsc.com/product-detail/Tantalum-Capacitors_Kyocera-AVX-TAJC107M016RNJ_C68621.html"
+			(at 233.68 105.41 0)
+			(effects
+				(font
+					(size 1.27 1.27)
+				)
+				(hide yes)
+			)
+		)
 		(pin "1"
 		)
@@
 			)
 		)
-		(property "Order" "https://www.mouser.vn/ProductDetail/Pulse-Electronics/PA4321.333NLT?qs=JxQonD1Dq%252BKcOFQkMu6Ckg%3D%3D"
+		(property "Order" "https://lcsc.com/product-detail/image/CYA0650-33UH_C5189937.html"
 			(at 223.52 101.6 0)
 			(effects
@@
 			)
 		)
-		(property "Value" "330uF/35V"
+		(property "Value" "100uF/16V"
 			(at 251.46 147.7009 0)
 			(effects
@@
 			)
 		)
-		(property "Footprint" "Capacitor_Tantalum_SMD:CP_EIA-3216-10_Kemet-I"
+		(property "Footprint" "Capacitor_Tantalum_SMD:CP_EIA-6032-15_Kemet-U"
 			(at 248.6152 151.13 0)
 			(effects
@@
 			)
 		)
+		(property "Order" "https://lcsc.com/product-detail/Tantalum-Capacitors_Kyocera-AVX-TAJC107M016RNJ_C68621.html"
+			(at 247.65 147.32 0)
+			(effects
+				(font
+					(size 1.27 1.27)
+				)
+				(hide yes)
+			)
+		)
 		(pin "2"
 		)
@@
 			)
 		)
+		(property "Order" "https://lcsc.com/product-detail/Tantalum-Capacitors_Kyocera-AVX-TAJC107M016RNJ_C68621.html"
+			(at 157.48 45.72 0)
+			(effects
+				(font
+					(size 1.27 1.27)
+				)
+				(hide yes)
+			)
+		)
 		(pin "1"
 		)
@@
 			)
 		)
-		(property "Value" "330uF/16V"
+		(property "Value" "100uF/16V"
 			(at 161.29 95.6309 0)
 			(effects
@@
 			)
 		)
+		(property "Order" "https://lcsc.com/product-detail/Tantalum-Capacitors_Kyocera-AVX-TAJC107M016RNJ_C68621.html"
+			(at 157.48 95.25 0)
+			(effects
+				(font
+					(size 1.27 1.27)
+				)
+				(hide yes)
+			)
+		)
 		(pin "1"
 		)
@@
 			)
 		)
-		(property "Value" "330uF/16V"
+		(property "Value" "100uF/16V"
 			(at 147.32 142.6209 0)
 			(effects
@@
 			)
 		)
+		(property "Order" "https://lcsc.com/product-detail/Tantalum-Capacitors_Kyocera-AVX-TAJC107M016RNJ_C68621.html"
+			(at 143.51 142.24 0)
+			(effects
+				(font
+					(size 1.27 1.27)
+				)
+				(hide yes)
+			)
+		)
 		(pin "1"
 		)
@@
 			)
 		)
-		(property "Order" "https://www.mouser.vn/ProductDetail/Pulse-Electronics/PA4321.333NLT?qs=JxQonD1Dq%252BKcOFQkMu6Ckg%3D%3D"
+		(property "Order" "https://lcsc.com/product-detail/image/CYA0650-33UH_C5189937.html"
 			(at 220.98 143.51 0)
 			(effects
@@
 			)
 		)
+		(property "Order" "https://lcsc.com/product-detail/image/CY2103MD1IEF4CC2A8_C2761719.html"
+			(at 43.18 66.04 0)
+			(effects
+				(font
+					(size 1.27 1.27)
+				)
+				(hide yes)
+			)
+		)
 		(pin "1"
 		)
@@
 			)
 		)
-		(property "Order" "https://www.mouser.vn/ProductDetail/Texas-Instruments/MC34063AD?qs=paYhMW8qfiu9F0uJ%2FIS%252Baw%3D%3D&srsltid=AfmBOoq7SQ5QFw4yrQjWeq76Xpg9N_VuEEG-eT88aM5SsiQV-1PSF91b"
+		(property "Order" "https://lcsc.com/product-detail/image/MC34063ADR_C100023.html"
 			(at 201.93 96.52 0)
 			(effects
