File: Charger_MPPT/Board_MPPT_40Az.kicad_pcb (KiCad board)
At the start: 2 copper layers, 195.4 x 117.6 mm, 359 parts, among them J1 USB_B_Micro, J10 RJ45_LED_Shielded, J11 Conn_01x02, J12 Conn_01x02, J13 Conn_01x02, J15 PJ012-8P8C1, J16 Conn_01x09_Pin, J19 LCD16x2_I2C, J2 1932768-1, J3 NMJ6HCD2, J4 Conn_01x02, J5 Conn_01x02, J6 NTC, J7 Conn_01x03_Pin, J8 Conn_01x06_Pin, J9 ID09S33E4GV00LF, Q1 2N7002, Q10 IPD053N08N3GATMA1, Q11 IPD053N08N3GATMA1, Q12 BC847, Q13 IRF740, Q14 IPD053N08N3GATMA1, Q15 BC847, Q16 DMP3028LFD, Q2 DMG1012T, Q3 2N7002, Q4 DMG1012T, Q6 BC847, Q7 IPD053N08N3GATMA1, Q8 IPD053N08N3GATMA1, Q9 IPD053N08N3GATMA1, SW1 SW_Push, U1 NXB0104PWJ, U10 ENC28J60/SS, U11 MCP1799T-3302H/DB, U16 LMV321, U2 GPS GNSS LC86L Quectel, U23 SP3485EN-L/TR, U24 SP3485EN-L/TR, U25 FS8205, U26 DS3231M, U27 DW01A, U28 MC34063AD, U29 AP62200, U3 Quectel_EC800M_CNGC-I03-SNNDA, U31 HLSR 80-P/SP10, U33 LM5017SD, U34 NCP5183DR2G, U35 NCP5183DR2G, U36 LMV321, U37 HLSR_50-P_SP33, U4 STM32F407VETx, U5 ESP32-WROOM-32UE-N4, U6 74HC14, U7 74HC14, U8 MAX3232, U9 LM2596S-5, Y1 8MHZ, Y2 25MHz

Commit message: added order link
Parts:
- C112: value 100uF/25V -> 100uF/16V; footprint Capacitor_Tantalum_SMD:CP_EIA-7343-43_Kemet-X -> Capacitor_Tantalum_SMD:CP_EIA-6032-20_AVX-F_Pad2.25x2.35mm_HandSolder
- C115: value 330uF/35V -> 100uF/16V; footprint Capacitor_Tantalum_SMD:CP_EIA-3216-10_Kemet-I -> Capacitor_Tantalum_SMD:CP_EIA-6032-15_Kemet-U
- C32, C34: value 330uF/16V -> 100uF/16V
- moved C113 1.29 mm to (188.4, 69.7)
- moved C115 1.09 mm to (191.6, 68.5)
Connections:
- net BAT + renamed +12P
Routing:
- net GND: track 0.00 -> 2.36 mm, vias 884 -> 886
- net /INTERFACE/interface.mb_tx: track 65.5 -> 63.8 mm
- net +3V3: track 396.2 -> 395.5 mm
- net Net-(C3-Pad1): vias 3 -> 2
Other:
- board text added: "0V"
- board text added: "BAT"
- board text added: "INPUT"
- board text added: "SWC"
- board text added: "SWD"

Commit message: added order link
Parts:
- C132, C43: value 4700uF/250V -> 330uF/160V
- C143, C144, C145, C146, C147, C44: value 330uF/250 -> 330uF/160
- F4: value Fuse -> 32v/60A
- moved D3 0.16 mm to (195.8, 35.4)
- moved R1 0.16 mm to (192.2, 35.5)
Connections:
- net +12P renamed BAT +
- C140 pad 1: /MPPT_70A/VCC12V -> +12V
- C141 pad 1: /MPPT_70A/VCC12V -> +12V
- C142 pad 1: /MPPT_70A/VCC12V -> +12V
- C150 pad 1: /MPPT_70A/VCC12V -> +12V
- D16 pad 2: /MPPT_70A/VCC12V -> +12V
- L5 pad 2: /MPPT_70A/VCC12V -> +12V
- R145 pad 1: /MPPT_70A/VCC12V -> +12V
- R54 pad 2: /MPPT_70A/VCC12V -> +12V
- R59 pad 1: /MPPT_70A/VCC12V -> +12V
- R75 pad 1: /MPPT_70A/VCC12V -> +12V
- U34 pad 5: /MPPT_70A/VCC12V -> +12V
- U35 pad 5: /MPPT_70A/VCC12V -> +12V
Routing:
- net /MPPT_70A/VCC12V: track 49.8 -> 0.00 mm, vias 21 -> 0
- net +12V: track 28.8 -> 55.0 mm, vias 0 -> 30
- net +3V3: track 395.5 -> 396.5 mm
- net GND: track 2.36 -> 2.99 mm, vias 886 -> 897
- added copper zone on B.Cu, net +12V
- removed copper zone on B.Cu, net /MPPT_70A/VCC12V
- removed copper zone on F.Cu, net /MPPT_70A/VCC12V
Other:
- outline, holes or cut-outs redrawn
- board text added: "+"
- board text added: "-"
- board text added: "3V3"
- board text added: "5V"
- board text added: "ADC"
- board text added: "CLK"
- board text added: "DC"
- board text added: "EN"
- board text added: "FAN"
- board text added: "GP0"
- board text added: "GPS"
- board text added: "MAIN"
- board text added: "MISO"
- board text added: "MOSI"
- board text added: "NTC"
- board text added: "RESET"
- board text added: "RST_L"
- board text added: "RX"
- board text added: "RX0"
- board text added: "SCL"
- board text added: "SDA"
- board text added: "SS"
- board text added: "TX"
- board text added: "TX0"
