File: Charger_MPPT/Board_MPPT_40Az.kicad_sch (KiCad schematic)
At the start: 6 parts

Commit message: added order link
Changed lines of the file:
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@@
+	(wire
+		(pts
+			(xy 176.53 59.69) (xy 176.53 54.61)
+		)
+		(stroke
+			(width 0)
+			(type default)
+		)
+	)
 	(wire
 		(pts
@@
 	(wire
 		(pts
+			(xy 180.34 54.61) (xy 180.34 50.8)
+		)
+		(stroke
+			(width 0)
+			(type default)
+		)
+	)
+	(wire
+		(pts
 			(xy 177.8 68.58) (xy 175.26 68.58)
 		)
@@
 	(wire
 		(pts
+			(xy 177.8 59.69) (xy 176.53 59.69)
+		)
+		(stroke
+			(width 0)
+			(type default)
+		)
+	)
+	(wire
+		(pts
 			(xy 138.43 62.23) (xy 134.62 62.23)
 		)
@@
 		(pts
 			(xy 135.89 53.34) (xy 138.43 53.34)
+		)
+		(stroke
+			(width 0)
+			(type default)
+		)
+	)
+	(wire
+		(pts
+			(xy 176.53 54.61) (xy 180.34 54.61)
 		)
 		(stroke
@@
 		)
 		(pin "+12V" input
-			(at 121.92 45.72 180)
-			(effects
-				(font
+			(at 180.34 50.8 270)
+			(effects
+				(font

Commit message: final link order
Parts:
- R78, R79, R80, R81, R82, R83: Order (none) -> https://lcsc.com/product-detail/image/FRC1206P000-TS_C29074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
Changed lines of the file:
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@@
+			)
+		)
+		(property "Order" "https://lcsc.com/product-detail/image/FRC1206P000-TS_C2907406.html"
+			(at 102.87 91.44 90)
+			(effects
+				(font
+					(size 1.27 1.27)
+				)
+				(hide yes)
 			)
 		)
@@
 			)
 		)
+		(property "Order" "https://lcsc.com/product-detail/image/FRC1206P000-TS_C2907406.html"
+			(at 123.19 91.44 90)
+			(effects
+				(font
+					(size 1.27 1.27)
+				)
+				(hide yes)
+			)
+		)
 		(pin "1"
 		)
@@
 			)
 		)
+		(property "Order" "https://lcsc.com/product-detail/image/FRC1206P000-TS_C2907406.html"
+			(at 102.87 109.22 90)
+			(effects
+				(font
+					(size 1.27 1.27)
+				)
+				(hide yes)
+			)
+		)
 		(pin "1"
 		)
@@
 			)
 		)
+		(property "Order" "https://lcsc.com/product-detail/image/FRC1206P000-TS_C2907406.html"
+			(at 123.19 100.33 90)
+			(effects
+				(font
+					(size 1.27 1.27)
+				)
+				(hide yes)
+			)
+		)
 		(pin "1"
 		)
@@
 			)
 		)
+		(property "Order" "https://lcsc.com/product-detail/image/FRC1206P000-TS_C2907406.html"
+			(at 123.19 109.22 90)
+			(effects
+				(font
+					(size 1.27 1.27)
+				)
+				(hide yes)
+			)
+		)
 		(pin "1"
 		)
@@
 			(effects
 				(font
+					(size 1.27 1.27)
+				)
+				(hide yes)
+			)
+		)
+		(property "Order" "https://lcsc.com/product-detail/image/FRC1206P000-TS_C2907406.html"
+			(at 102.87 100.33 90)
+			(effects
+				(font
