File: Charger_MPPT/MCU.kicad_sch (KiCad schematic)
At the start: 37 parts, among them J16 Conn_01x09_Pin, J7 Conn_01x03_Pin, J8 Conn_01x06_Pin, Q15 BC847, SW1 SW_Push, U4 STM32F407VETx, U5 ESP32-WROOM-32UE-N4, Y1 8MHZ

Commit message: added order link
Parts:
- Q15: Order (none) -> https://www.lcsc.com/product-detail/Bipolar-BJT_Nexperia-BC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
- U4: Order https://www.mouser.vn/ProductDetail/STMicroelectronics/STM3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 -> https://lcsc.com/product-detail/image/STM32F407VET6TR_C5269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
- U5: Order https://www.mouser.vn/ProductDetail/Espressif-Systems/ESP32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 -> https://lcsc.com/product-detail/image/ESP32-WROOM-32UE-N4_C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
- Y1: Order https://www.mouser.vn/ProductDetail/ECS/ECS-080-18-23G-JGN-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 -> https://lcsc.com/product-detail/image/X50328MSB2GI_C115962.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
Changed lines of the file:
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@@
 			)
 		)
-		(property "Order" "https://www.mouser.vn/ProductDetail/STMicroelectronics/STM32F407VET6?qs=Z8%252BeY1k3TIJFAMMqSR%252BGtw%3D%3D&srsltid=AfmBOopnDMgfPflhfQg0FdQOsn5CCJbP6Kq-wiVHECpvvzL41hgnXbeO"
+		(property "Order" "https://lcsc.com/product-detail/image/STM32F407VET6TR_C5269943.html"
 			(at 200.66 275.59 0)
 			(effects
@@
 			)
 		)
-		(property "Order" "https://www.mouser.vn/ProductDetail/Espressif-Systems/ESP32-WROOM-32UE-N4?qs=Li%252BoUPsLEnsnnWrvUBU2ZA%3D%3D"
+		(property "Order" "https://lcsc.com/product-detail/image/ESP32-WROOM-32UE-N4_C701344.html"
 			(at 199.39 133.35 0)
 			(effects
@@
 			)
 		)
-		(property "Order" "https://www.mouser.vn/ProductDetail/ECS/ECS-080-18-23G-JGN-TR?qs=HXFqYaX1Q2w96I4MjMnYbA%3D%3D"
+		(property "Order" "https://lcsc.com/product-detail/image/X50328MSB2GI_C115962.html"
 			(at 66.04 248.92 0)
 			(effects
@@
 			(at 81.28 318.77 0)
 			(effects
+				(font
+					(size 1.27 1.27)
+				)
+				(hide yes)
+			)
+		)
+		(property "Order" "https://www.lcsc.com/product-detail/Bipolar-BJT_Nexperia-BC847B-215_C57668.html?s_z=n_BC847"
+			(at 81.28 318.77 0)
+			(effects

Commit message: final link order
Parts:
- SW1: Order (none) -> https://lcsc.com/product-detail/image/TS-1101-C-W_C318938.h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
Changed lines of the file:
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@@
+			)
+		)
+		(property "Order" "https://lcsc.com/product-detail/image/TS-1101-C-W_C318938.html"
+			(at 134.62 212.09 0)
+			(effects
+				(font
+					(size 1.27 1.27)
+				)
+				(hide yes)
 			)
 		)
