File: Charger_MPPT/MPPT_70A.kicad_sch (KiCad schematic)
At the start: 108 parts, among them J11 Conn_01x02, J4 Conn_01x02, J5 Conn_01x02, J6 NTC, Q10 IPD053N08N3GATMA1, Q11 IPD053N08N3GATMA1, Q12 BC847, Q13 IRF740, Q14 IPD053N08N3GATMA1, Q7 IPD053N08N3GATMA1, Q8 IPD053N08N3GATMA1, Q9 IPD053N08N3GATMA1, U16 LMV321, U31 HLSR 80-P/SP10, U33 LM5017SD, U34 NCP5183DR2G, U35 NCP5183DR2G, U36 LMV321, U37 HLSR_50-P_SP33

Commit message: added order link
Parts:
- J4: Order (none) -> https://lcsc.com/product-detail/image/WJ55C-B-10-0-2P_C4602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
Changed lines of the file:
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@@
+			)
+		)
+		(property "Order" "https://lcsc.com/product-detail/image/WJ55C-B-10-0-2P_C46028.html"
+			(at 33.02 22.86 0)
+			(effects
+				(font
+					(size 1.27 1.27)
+				)
+				(hide yes)
 			)
 		)

Commit message: added order link
Parts:
- D15: Order (none) -> https://lcsc.com/product-detail/image/MBR0520_C5204745.html
- F4: value Fuse -> 32v/60A; Order (none) -> https://lcsc.com/product-detail/image/0299060-ZXNV_C178945.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
- Q7: Order (none) -> https://www.mouser.com/ProductDetail/Infineon-Technologies/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
Changed lines of the file:
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@@
 			)
 		)
-		(property "Value" "Fuse"
+		(property "Value" "32v/60A"
 			(at 26.67 29.21 90)
 			(effects
@@
 		(property "Description" ""
 			(at 26.67 31.75 0)
+			(effects
+				(font
+					(size 1.27 1.27)
+				)
+				(hide yes)
+			)
+		)
+		(property "Order" "https://lcsc.com/product-detail/image/0299060-ZXNV_C178945.html"
+			(at 26.67 31.75 90)
 			(effects
 				(font
@@
 			)
 		)
+		(property "Order" "https://www.mouser.com/ProductDetail/Infineon-Technologies/IPD053N08N3GATMA1?qs=3Bi3m9r5MQbqPBHFEv2uTQ%3D%3D&srsltid=AfmBOoqBrUTgscBYnOP4M8PfFPxqnfI-XQ4hNAr7mChqfNOpxYw-ShdW"
+			(at 33.02 59.69 0)
+			(effects
+				(font
+					(size 1.27 1.27)
+				)
+				(hide yes)
+			)
+		)
 		(pin "2"
 		)
@@
 			(effects
 				(font
+					(size 1.27 1.27)
+				)
+				(hide yes)
+			)
+		)
+		(property "Order" "https://lcsc.com/product-detail/image/MBR0520_C5204745.html"
+			(at 44.45 63.5 90)
+			(effects
+				(font

Commit message: added order link
Parts:
- C132, C43: value 4700uF/250V -> 330uF/160V; Order (none) -> https://lcsc.com/product-detail/image/EKXJ161ELL331MLN3S_C7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
- C139, C151: Order (none) -> https://lcsc.com/product-detail/image/NM1206B474K201CEGN_C7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
- C143, C144, C145, C146, C147, C44: value 330uF/250 -> 330uF/160; Order (none) -> https://lcsc.com/product-detail/image/EKXJ161ELL331MLN3S_C7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
- D18, D19: Order (none) -> https://lcsc.com/product-detail/image/SS210_C488408.html
- Q10, Q11, Q8, Q9: Order (none) -> https://www.mouser.com/ProductDetail/Infineon-Technologies/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
- R143, R148, R149, R61, R63: Order (none) -> https://www.lcsc.com/product-detail/Chip-Resistor-Surface-M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
- R145, R146, R147, R59, R60, R62: Order (none) -> https://lcsc.com/product-detail/image/FRC0805F2R40TS_C29303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
- R150, R58: Order (none) -> https://lcsc.com/product-detail/image/FRP2512F0000TS_C52040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
- R49: Order (none) -> https://lcsc.com/product-detail/image/RC0805FR-07100KL_C963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
- R50: Order (none) -> https://lcsc.com/product-detail/image/0805W8F5601T5E_C4382.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
- R56, R57, R64, R65: Order (none) -> https://lcsc.com/product-detail/image/0805W8F1000T5E_C17408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
- U31: Order (none) -> https://www.digikey.com/en/products/detail/lem-usa-inc/HLSR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
- U34: Order (none) -> https://lcsc.com/product-detail/Gate-Drivers_onsemi-NCP5183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

Commit message: added order link
Parts:
- C46: value 100uF/25V -> 10uF/25V; Order (none) -> https://lcsc.com/product-detail/image/T491A106K016AT_C11005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
- J11: Order (none) -> https://lcsc.com/product-detail/Barrier-Terminal-Blocks_TE-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
- J4: Order https://lcsc.com/product-detail/image/WJ55C-B-10-0-2P_C4602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 -> https://lcsc.com/product-detail/Barrier-Terminal-Blocks_TE-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; Order1 (none) -> https://lcsc.com/product-detail/Barrier-Terminal-Blocks_TE-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
- J5, J6: Order (none) -> https://lcsc.com/product-detail/image/B2B-XH-A-LF-SN_C15801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
- Q13: Order (none) -> https://lcsc.com/product-detail/image/IRF740_C358408.html
- Q14: Order (none) -> https://www.mouser.com/ProductDetail/Infineon-Technologies/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
- R151, R68, R70: Order (none) -> https://lcsc.com/product-detail/image/0805W8F1000T5E_C17408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
- R152, R71: Order (none) -> https://lcsc.com/product-detail/image/RC0805FR-071KL_C95781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
- R153, R72: Order (none) -> https://lcsc.com/product-detail/image/RC0805FR-0730KL_C1263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
- R66, R76: Order (none) -> https://www.lcsc.com/product-detail/Chip-Resistor-Surface-M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
- R67, R69: Order (none) -> https://lcsc.com/product-detail/image/0805W8F2201T5E_C17520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
- R73: Order (none) -> https://lcsc.com/product-detail/image/0805W8F8202T5E_C17840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
- R74, R75: Order (none) -> https://lcsc.com/product-detail/image/RC0805FR-0710KL_C8437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
- U16, U36: Order (none) -> https://lcsc.com/product-detail/image/LMV321IDBVR_C7972.html
- U35: Order (none) -> https://lcsc.com/product-detail/Gate-Drivers_onsemi-NCP5183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
- U37: Order (none) -> https://www.digikey.com/en/products/detail/lem-usa-inc/HLSR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
Changed lines of the file:
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@@
 			)
 		)
+		(property "Order" "https://lcsc.com/product-detail/image/LMV321IDBVR_C7972.html"
+			(at 474.98 107.95 0)
+			(effects
+				(font
+					(size 1.27 1.27)
+				)
+				(hide yes)
+			)
+		)
 		(pin "3"
 		)
@@
 			)
 		)
+		(property "Order" "https://www.lcsc.com/product-detail/Chip-Resistor-Surface-Mount_YAGEO-AC0805FR-7W10KL_C855098.html?s_z=n_10k"
+			(at 66.04 219.71 0)
+			(effects
+				(font
+					(size 1.27 1.27)
+				)
+				(hide yes)
+			)
+		)
 		(pin "1"
 		)
@@
 			)
 		)
+		(property "Order" "https://lcsc.com/product-detail/image/RC0805FR-0730KL_C126352.html"
+			(at 483.87 118.11 90)
+			(effects
+				(font
+					(size 1.27 1.27)
+				)
+				(hide yes)
+			)
+		)
 		(pin "1"
 		)
@@
 			)
 		)
+		(property "Order" "https://lcsc.com/product-detail/image/0805W8F8202T5E_C17840.html"
+			(at 128.27 149.86 0)
+			(effects
+				(font
+					(size 1.27 1.27)
+				)
+				(hide yes)
+			)
+		)
 		(pin "1"
 		)
@@
 			)
 		)
+		(property "Order" "https://lcsc.com/product-detail/image/RC0805FR-0730KL_C126352.html"
+			(at 397.51 118.11 90)
+			(effects
+				(font
+					(size 1.27 1.27)
+				)
+				(hide yes)
+			)
+		)
 		(pin "1"
 		)
@@
 			)
 		)
+		(property "Order" "https://lcsc.com/product-detail/Barrier-Terminal-Blocks_TE-Connectivity-6PCV-02-006_C3656257.html?s_z=n_6PCV-02-006"
+			(at 165.1 176.53 0)
+			(effects
+				(font
+					(size 1.27 1.27)
+				)
+				(hide yes)
+			)
+		)
 		(pin "1"
 		)
@@
 		)
 		(property "Value" "100R"
-			(at 381 165.1 90)
+			(at 380.746 167.64 90)
 			(effects
 				(font
@@
 			)
 		)
+		(property "Order" "https://lcsc.com/product-detail/image/0805W8F1000T5E_C17408.html"
+			(at 381 167.64 90)
+			(effects
+				(font
+					(size 1.27 1.27)
+				)
+				(hide yes)
+			)
+		)
 		(pin "1"
 		)
@@
 				)
 				(justify left)
-				(hide yes)
 			)
 		)
@@
 			)
 		)
+		(property "Order" "https://www.mouser.com/ProductDetail/Infineon-Technologies/IPD053N08N3GATMA1?qs=3Bi3m9r5MQbqPBHFEv2uTQ%3D%3D&srsltid=AfmBOoqBrUTgscBYnOP4M8PfFPxqnfI-XQ4hNAr7mChqfNOpxYw-ShdW"
+			(at 99.06 201.93 0)
+			(effects
+				(font
+					(size 1.27 1.27)
+				)
+				(hide yes)
+			)
+		)
 		(pin "2"
 		)
@@
 			)
 		)
-		(property "Order" "https://lcsc.com/product-detail/image/WJ55C-B-10-0-2P_C46028.html"
+		(property "Order" "https://lcsc.com/product-detail/Barrier-Terminal-Blocks_TE-Connectivity-6PCV-02-006_C3656257.html?s_z=n_6PCV-02-006"
+			(at 33.02 22.86 0)
+			(effects
+				(font
+					(size 1.27 1.27)
+				)
+				(hide yes)
+			)
+		)
+		(property "Order1" "https://lcsc.com/product-detail/Barrier-Terminal-Blocks_TE-Connectivity-6PCV-02-006_C3656257.html?s_z=n_6PCV-02-006"
 			(at 33.02 22.86 0)
 			(effects
@@
 			)
 		)
-		(property "Value" "100uF/25V"
+		(property "Value" "10uF/25V"
 			(at 394.97 194.6909 0)
 			(effects
@@
 			)
 		)
+		(property "Order" "https://lcsc.com/product-detail/image/T491A106K016AT_C110055.html"
+			(at 391.16 194.31 0)
+			(effects
+				(font
+					(size 1.27 1.27)
+				)
+				(hide yes)
+			)
+		)
 		(pin "1"
 		)
@@
 		(dnp no)
 		(property "Reference" "R66"
-			(at 384.81 212.09 90)
+			(at 388.366 212.09 90)
 			(effects
 				(font
@@
 		)
 		(property "Value" "10k"
-			(at 393.7 212.09 90)
+			(at 391.16 212.09 90)
 			(effects
 				(font
@@
 			)
 		)
+		(property "Order" "https://www.lcsc.com/product-detail/Chip-Resistor-Surface-Mount_YAGEO-AC0805FR-7W10KL_C855098.html?s_z=n_10k"
+			(at 391.16 212.09 90)
+			(effects
+				(font
+					(size 1.27 1.27)
+				)
+				(hide yes)
+			)
+		)
 		(pin "1"
 		)
@@
 			)
 		)
+		(property "Order" "https://lcsc.com/product-detail/image/RC0805FR-0710KL_C84376.html"
+			(at 74.93 195.58 0)
+			(effects
+				(font
+					(size 1.27 1.27)
+				)
+				(hide yes)
+			)
+		)
 		(pin "1"
 		)
@@
 			)
 		)
+		(property "Order" "https://lcsc.com/product-detail/image/0805W8F1000T5E_C17408.html"
+			(at 454.66 101.6 90)
+			(effects
+				(font
+					(size 1.27 1.27)
+				)
+				(hide yes)
+			)
+		)
 		(pin "1"
 		)
@@
 			)
 		)
+		(property "Order" "https://lcsc.com/product-detail/image/B2B-XH-A-LF-SN_C158012.html"
+			(at 364.49 193.04 0)
+			(effects
+				(font
+					(size 1.27 1.27)
+				)
+				(hide yes)
+			)
+		)
 		(pin "1"
 		)
@@
 		(dnp no)
 		(property "Reference" "R67"
-			(at 402.59 212.09 90)
+			(at 402.59 208.534 90)
 			(effects
 				(font
@@
 		)
 		(property "Value" "2k2"
-			(at 402.59 203.2 90)
+			(at 402.336 205.74 90)
 			(effects
 				(font
@@
 			)
 		)
+		(property "Order" "https://lcsc.com/product-detail/image/0805W8F2201T5E_C17520.html"
+			(at 402.59 205.74 90)
+			(effects
+				(font
+					(size 1.27 1.27)
+				)
+				(hide yes)
+			)
+		)
 		(pin "1"
 		)
@@
 			)
 		)
+		(property "Order" "https://lcsc.com/product-detail/image/RC0805FR-0710KL_C84376.html"
+			(at 128.27 170.18 0)
+			(effects
+				(font
+					(size 1.27 1.27)
+				)
+				(hide yes)
+			)
+		)
 		(pin "1"
 		)
@@
 			)
 		)
+		(property "Order" "https://lcsc.com/product-detail/image/RC0805FR-071KL_C95781.html"
+			(at 375.92 121.92 90)
+			(effects
+				(font
+					(size 1.27 1.27)
+				)
+				(hide yes)
+			)
+		)
 		(pin "1"
 		)
@@
 			)
 		)
+		(property "Order" "https://lcsc.com/product-detail/image/IRF740_C358408.html"
+			(at 378.46 205.74 0)
+			(effects
+				(font
+					(size 1.27 1.27)
+				)
+				(hide yes)
+			)
+		)
 		(pin "2"
 		)
@@
 			)
 		)
+		(property "Order" "https://lcsc.com/product-detail/image/0805W8F1000T5E_C17408.html"
+			(at 368.3 101.6 90)
+			(effects
+				(font
+					(size 1.27 1.27)
+				)
+				(hide yes)
+			)
+		)
 		(pin "1"
 		)
@@
 			)
 		)
+		(property "Order" "https://lcsc.com/product-detail/Gate-Drivers_onsemi-NCP5183DR2G_C904511.html?s_z=n_NCP5183DR2G"
+			(at 242.57 140.97 0)
+			(effects
+				(font
+					(size 1.27 1.27)
+				)
+				(hide yes)
+			)
+		)
 		(pin "4"
 		)
@@
 			)
 		)
+		(property "Order" "https://www.digikey.com/en/products/detail/lem-usa-inc/HLSR-50-P/4331982"
+			(at 64.77 163.83 90)
+			(effects
+				(font
+					(size 1.27 1.27)
+				)
+				(hide yes)
+			)
+		)
 		(pin "7"
 		)
@@
 			)
 		)
+		(property "Order" "https://lcsc.com/product-detail/image/RC0805FR-071KL_C95781.html"
+			(at 462.28 121.92 90)
+			(effects
+				(font
+					(size 1.27 1.27)
+				)
+				(hide yes)
+			)
+		)
 		(pin "1"
 		)
@@
 			)
 		)
+		(property "Order" "https://lcsc.com/product-detail/image/B2B-XH-A-LF-SN_C158012.html"
+			(at 364.49 170.18 0)
+			(effects
+				(font
+					(size 1.27 1.27)
+				)
+				(hide yes)
+			)
+		)
 		(pin "1"
 		)
@@
 			)
 		)
+		(property "Order" "https://lcsc.com/product-detail/image/LMV321IDBVR_C7972.html"
+			(at 388.62 107.95 0)
+			(effects
+				(font
+					(size 1.27 1.27)
+				)
+				(hide yes)
+			)
+		)
 		(pin "3"
 		)
@@
 		)
 		(property "Value" "2k2"
-			(at 369.57 162.56 90)
+			(at 372.11 162.814 90)
 			(effects
 				(font
@@
 			(effects
 				(font
+					(size 1.27 1.27)
+				)
+				(hide yes)
+			)
+		)
+		(property "Order" "https://lcsc.com/product-detail/image/0805W8F2201T5E_C17520.html"
+			(at 372.11 162.56 90)
+			(effects
+				(font

Commit message: final link order
Parts:
- C141: Order (none) -> https://lcsc.com/product-detail/image/TAJA475K025RNJ_C7189.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
- C70, C71: Order (none) -> https://www.lcsc.com/product-detail/Multilayer-Ceramic-Capa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
- D16: Order (none) -> https://lcsc.com/product-detail/Switching-Diodes_VISHAY-1N4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
- L5: Order (none) -> https://lcsc.com/product-detail/image/SLH0704S221MTT_C49241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
- PS1: Order (none) -> https://lcsc.com/product-detail/image/B0505S-1WR3_C7465178.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
- Q12: Order (none) -> https://lcsc.com/product-detail/image/BC847B-215_C57668.html
- R144: Order (none) -> https://lcsc.com/product-detail/image/RC0805FR-0710KL_C8437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
- R48: Order (none) -> https://lcsc.com/product-detail/image/1206W4F1002T5E_C17902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
- R51: Order (none) -> https://lcsc.com/product-detail/image/RT0805BRD0791KL_C8657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
- R52, R55: Order (none) -> https://www.lcsc.com/product-detail/Chip-Resistor-Surface-M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
- R53: Order (none) -> https://lcsc.com/product-detail/image/FRC0805F4993TS_C29609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
- R54: Order (none) -> https://lcsc.com/product-detail/image/RT0805BRD0788K7L_C706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
- R77: Order (none) -> https://lcsc.com/product-detail/image/0805W8F1000T5E_C17408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
- U33: Order (none) -> https://www.mouser.vn/ProductDetail/Texas-Instruments/LM501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
Changed lines of the file:
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@@
 			)
 		)
+		(property "Order" "https://lcsc.com/product-detail/Switching-Diodes_VISHAY-1N4148W-E3-08_C241939.html?s_z=n_1N4148W"
+			(at 137.16 120.65 0)
+			(effects
+				(font
+					(size 1.27 1.27)
+				)
+				(hide yes)
+			)
+		)
 		(pin "2"
 		)
@@
 			)
 		)
+		(property "Order" "https://www.mouser.vn/ProductDetail/Texas-Instruments/LM5017SD-NOPB?qs=iiglMaU8SAdQJx7ZXr%252BBlQ%3D%3D&srsltid=AfmBOooXXU3ASupGjZuKDGf3qDGLZvltX6rVMSK2fyLZUJVy21tiRzF-"
+			(at 97.79 113.03 0)
+			(effects
+				(font
+					(size 1.27 1.27)
+				)
+				(hide yes)
+			)
+		)
 		(pin "3"
 		)
@@
 			)
 		)
+		(property "Order" "https://www.lcsc.com/product-detail/Chip-Resistor-Surface-Mount_YAGEO-AC0805FR-7W10KL_C855098.html?s_z=n_10k"
+			(at 43.18 123.19 0)
+			(effects
+				(font
+					(size 1.27 1.27)
+				)
+				(hide yes)
+			)
+		)
 		(pin "1"
 		)
@@
 			)
 		)
+		(property "Order" "https://lcsc.com/product-detail/image/BC847B-215_C57668.html"
+			(at 72.39 208.28 0)
+			(effects
+				(font
+					(size 1.27 1.27)
+				)
+				(hide yes)
+			)
+		)
 		(pin "3"
 		)
@@
 			)
 		)
+		(property "Order" "https://lcsc.com/product-detail/image/TAJA475K025RNJ_C7189.html"
+			(at 151.13 124.46 0)
+			(effects
+				(font
+					(size 1.27 1.27)
+				)
+				(hide yes)
+			)
+		)
 		(pin "1"
 		)
@@
 			)
 		)
+		(property "Order" "https://lcsc.com/product-detail/image/FRC0805F4993TS_C2960934.html"
+			(at 67.31 110.49 90)
+			(effects
+				(font
+					(size 1.27 1.27)
+				)
+				(hide yes)
+			)
+		)
 		(pin "1"
 		)
@@
 			)
 		)
+		(property "Order" "https://lcsc.com/product-detail/image/1206W4F1002T5E_C17902.html"
+			(at 44.45 43.18 0)
+			(effects
+				(font
+					(size 1.27 1.27)
+				)
+				(hide yes)
+			)
+		)
 		(pin "1"
 		)
@@
 			)
 		)
+		(property "Order" "https://lcsc.com/product-detail/image/RC0805FR-0710KL_C84376.html"
+			(at 85.09 179.07 0)
+			(effects
+				(font
+					(size 1.27 1.27)
+				)
+				(hide yes)
+			)
+		)
 		(pin "1"
 		)
@@
 			)
 		)
+		(property "Order" "https://www.lcsc.com/product-detail/Multilayer-Ceramic-Capacitors-MLCC-SMD-SMT_YAGEO-CC0805KRX7R9BB104_C49678.html"
+			(at 214.63 185.42 0)
+			(effects
+				(font
+					(size 1.27 1.27)
+				)
+				(hide yes)
+			)
+		)
 		(pin "1"
 		)
@@
 			)
 		)
+		(property "Order" "https://www.lcsc.com/product-detail/Chip-Resistor-Surface-Mount_YAGEO-AC0805FR-7W10KL_C855098.html?s_z=n_10k"
+			(at 124.46 128.27 0)
+			(effects
+				(font
+					(size 1.27 1.27)
+				)
+				(hide yes)
+			)
+		)
 		(pin "1"
 		)
@@
 			)
 		)
+		(property "Order" "https://www.lcsc.com/product-detail/Multilayer-Ceramic-Capacitors-MLCC-SMD-SMT_YAGEO-CC0805KRX7R9BB104_C49678.html"
+			(at 267.97 185.42 0)
+			(effects
+				(font
+					(size 1.27 1.27)
+				)
+				(hide yes)
+			)
+		)
 		(pin "1"
 		)
@@
 			)
 		)
+		(property "Order" "https://lcsc.com/product-detail/image/SLH0704S221MTT_C49241602.html"
+			(at 132.08 110.49 90)
+			(effects
+				(font
+					(size 1.27 1.27)
+				)
+				(hide yes)
+			)
+		)
 		(pin "1"
 		)
@@
 			)
 		)
+		(property "Order" "https://lcsc.com/product-detail/image/B0505S-1WR3_C7465178.html"
+			(at 241.3 184.15 0)
+			(effects
+				(font
+					(size 1.27 1.27)
+				)
+				(hide yes)
+			)
+		)
 		(pin "2"
 		)
@@
 			)
 		)
+		(property "Order" "https://lcsc.com/product-detail/image/RT0805BRD0788K7L_C706252.html"
+			(at 137.16 115.57 90)
+			(effects
+				(font
+					(size 1.27 1.27)
+				)
+				(hide yes)
+			)
+		)
 		(pin "1"
 		)
@@
 			)
 		)
+		(property "Order" "https://lcsc.com/product-detail/image/RT0805BRD0791KL_C865700.html"
+			(at 43.18 111.76 0)
+			(effects
+				(font
+					(size 1.27 1.27)
+				)
+				(hide yes)
+			)
+		)
 		(pin "1"
 		)
@@
 			(effects
 				(font
+					(size 1.27 1.27)
+				)
+				(hide yes)
+			)
+		)
+		(property "Order" "https://lcsc.com/product-detail/image/0805W8F1000T5E_C17408.html"
+			(at 62.23 208.28 90)
+			(effects
+				(font
