File: Charger_MPPT/PERIPHERAL.kicad_sch (KiCad schematic)
At the start: 67 parts, among them J1 USB_B_Micro, J2 1932768-1, J3 NMJ6HCD2, Q1 2N7002, Q2 DMG1012T, Q3 2N7002, Q4 DMG1012T, U1 NXB0104PWJ, U2 GPS GNSS LC86L Quectel, U3 Quectel_EC800M_CNGC-I03-SNNDA

Commit message: added order link
Parts:
- C15: Order https://www.digikey.com/en/products/detail/yageo/CC0805JRNP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 -> https://lcsc.com/product-detail/image/CC0603JRNPO9BN330_C10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
- J2: Order Avnet -> https://lcsc.com/product-detail/image/NANO-SIM-XG6P-H1-35_C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
- J3: Order (none) -> https://lcsc.com/product-detail/image/PJ-342_C668606.html
- Q2, Q4: Order https://www.mouser.vn/ProductDetail/Diodes-Incorporated/DMG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 -> https://lcsc.com/product-detail/image/DMG1012T-7_C20512.html
- U3: Link (none) -> https://www.alibaba.com/product-detail/Quectel-EC800M-CN-EC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
Changed lines of the file:
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@@
 			)
 		)
-		(property "Order" "https://www.mouser.vn/ProductDetail/Diodes-Incorporated/DMG1012T-7?qs=vIZ3oKQCLxoEnfyeB0HcGQ%3D%3D&srsltid=AfmBOoqRPLKHhD9PXrGb4mmYI4uEF9orsBisH3EDsfEf-Boy45JVQsqm"
+		(property "Order" "https://lcsc.com/product-detail/image/DMG1012T-7_C20512.html"
 			(at 124.46 204.47 0)
 			(effects
@@
 		(on_board yes)
 		(dnp no)
-		(fields_autoplaced yes)
 		(property "Reference" "C22"
-			(at 345.44 189.2299 0)
+			(at 334.01 184.912 0)
 			(effects
 				(font
@@
 		)
 		(property "Value" "10pF"
-			(at 345.44 191.7699 0)
+			(at 334.01 187.452 0)
 			(effects
 				(font
@@
 			)
 		)
+		(property "Link" "https://www.alibaba.com/product-detail/Quectel-EC800M-CN-EC800-Series-4G_1601266127333.html"
+			(at 289.56 166.37 0)
+			(effects
+				(font
+					(size 1.27 1.27)
+				)
+				(hide yes)
+			)
+		)
 		(pin "16"
 		)
@@
 			)
 		)
+		(property "Order" "https://lcsc.com/product-detail/image/PJ-342_C668606.html"
+			(at 392.43 175.26 0)
+			(effects
+				(font
+					(size 1.27 1.27)
+				)
+				(hide yes)
+			)
+		)
 		(pin "TN"
 		)
@@
 			)
 		)
-		(property "Order" "Avnet"
+		(property "Order" "https://lcsc.com/product-detail/image/NANO-SIM-XG6P-H1-35_C7529386.html"
 			(at 356.87 62.23 0)
 			(effects
@@
 			)
 		)
-		(property "Order" "https://www.mouser.vn/ProductDetail/Diodes-Incorporated/DMG1012T-7?qs=vIZ3oKQCLxoEnfyeB0HcGQ%3D%3D&srsltid=AfmBOoqRPLKHhD9PXrGb4mmYI4uEF9orsBisH3EDsfEf-Boy45JVQsqm"
+		(property "Order" "https://lcsc.com/product-detail/image/DMG1012T-7_C20512.html"
 			(at 59.69 204.47 0)
 			(effects
@@
 			)
 		)
-		(property "Order" "https://www.digikey.com/en/products/detail/yageo/CC0805JRNPO9BN330/302839"
+		(property "Order" "https://lcsc.com/product-detail/image/CC0603JRNPO9BN330_C107047.html"
 			(at 213.36 255.27 0)
 			(effects

Commit message: final link order
Parts:
- C12, C9: value NC -> 10nF; Order (none) -> https://lcsc.com/product-detail/image/GRM2195C1H103FA01D_C4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
- C3: Order https://www.lcsc.com/product-detail/Multilayer-Ceramic-Capa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 -> https://lcsc.com/product-detail/image/GRM2195C1H103FA01D_C4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
- C5, C8: value C -> 10nF; Order (none) -> https://lcsc.com/product-detail/image/GRM1885C1H103FA01D_C5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
Changed lines of the file:
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@@
 			)
 		)
-		(property "Order" "https://www.lcsc.com/product-detail/Multilayer-Ceramic-Capacitors-MLCC-SMD-SMT_YAGEO-CC0805KRX7R9BB103_C83170.html"
+		(property "Order" "https://lcsc.com/product-detail/image/GRM2195C1H103FA01D_C441760.html"
 			(at 62.23 266.7 0)
 			(effects
@@
 			)
 		)
-		(property "Value" "NC"
+		(property "Value" "10nF"
 			(at 163.068 263.144 0)
 			(effects
@@
 			)
 		)
-		(property "Order" ""
+		(property "Order" "https://lcsc.com/product-detail/image/GRM2195C1H103FA01D_C441760.html"
 			(at 158.75 260.35 0)
 			(effects
@@
 			)
 		)
-		(property "Value" "C"
+		(property "Value" "10nF"
 			(at 115.57 130.8099 0)
 			(effects
@@
 			)
 		)
+		(property "Order" "https://lcsc.com/product-detail/image/GRM1885C1H103FA01D_C5299898.html"
+			(at 111.76 129.54 0)
+			(effects
+				(font
+					(size 1.27 1.27)
+				)
+				(hide yes)
+			)
+		)
 		(pin "2"
 		)
@@
 			)
 		)
-		(property "Value" "C"
+		(property "Value" "10nF"
 			(at 92.71 130.8099 0)
 			(effects
@@
 			)
 		)
+		(property "Order" "https://lcsc.com/product-detail/image/GRM1885C1H103FA01D_C5299898.html"
+			(at 88.9 129.54 0)
+			(effects
+				(font
+					(size 1.27 1.27)
+				)
+				(hide yes)
+			)
+		)
 		(pin "2"
 		)
@@
 			)
 		)
-		(property "Value" "NC"
+		(property "Value" "10nF"
 			(at 128.778 263.144 0)
 			(effects
@@
 			)
 		)
-		(property "Order" ""
+		(property "Order" "https://lcsc.com/product-detail/image/GRM2195C1H103FA01D_C441760.html"
 			(at 124.46 260.35 0)
 			(effects
