File: Charger_MPPT/interface.kicad_sch (KiCad schematic)
At the start: 93 parts, among them J10 RJ45_LED_Shielded, J12 Conn_01x02, J13 Conn_01x02, J15 PJ012-8P8C1, J19 LCD16x2_I2C, J9 ID09S33E4GV00LF, U10 ENC28J60/SS, U11 MCP1799T-3302H/DB, U23 SP3485EN-L/TR, U24 SP3485EN-L/TR, U25 FS8205, U26 DS3231M, U27 DW01A, U6 74HC14, U7 74HC14, U8 MAX3232, Y2 25MHz

Commit message: added order link
Parts:
- BT1: Order https://giadungnhaviet.com/san-pham/pin-sac-cuc-ao-han-chan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 -> https://nshopvn.com/product/pin-sac-ni-mh/?variant=144643
- C87: Order (none) -> https://lcsc.com/product-detail/image/CL21A106KOQNNNE_C1713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
- D37, D38: Order (none) -> https://lcsc.com/product-detail/image/MHK2310RRBTD_C2764897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
- D39: Order (none) -> https://lcsc.com/product-detail/image/MBR0520_C5204745.html
- J10: Order (none) -> https://lcsc.com/product-detail/image/RJ45-334-053-01_C4734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
- J12, J13: Order (none) -> https://lcsc.com/product-detail/image/DB128V-5-08-2P-GN-S_C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
- J15: Order https://www.digikey.com/en/products/detail/on-shore-technol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 -> https://lcsc.com/product-detail/image/R-RJ45S08P-A004_C2902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
- J9: Order https://www.lcsc.com/product-detail/D-Sub-VGA-Connectors_Am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 -> https://lcsc.com/product-detail/D-Sub-VGA-Connectors_XUNPU-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
- U10: Order https://www.digikey.com/en/products/detail/microchip-techno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 -> https://lcsc.com/product-detail/image/ENC28J60-SS_C8961.html
- U11: Order https://www.mouser.vn/ProductDetail/Microchip-Technology/MC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 -> https://lcsc.com/product-detail/Voltage-Regulators-Linear-L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
- U23, U24: Order https://www.digikey.com/en/products/detail/maxlinear-inc/SP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 -> https://lcsc.com/product-detail/image/SP3485EN-L-TR_C8963.h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
- U25: Order https://www.amazon.ca/FS8205A-TSSOP8-FS8205-CEG8205A-CEG820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 -> https://icdayroi.com/fs8205a
- U26: Order https://www.mouser.vn/ProductDetail/Analog-Devices-Maxim-In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 -> https://lcsc.com/product-detail/image/DS3231SN-T-R_C9866.ht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
- U27: Order https://linhkienchatluong.vn/ic-nguon/dw01-sot23-6-ic-bao-v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 -> https://lcsc.com/product-detail/image/DW01A_C2927799.html
- Y2: Order https://www.mouser.vn/ProductDetail/CTS-Electronic-Componen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 -> https://lcsc.com/product-detail/image/X503225MSB2GI_C112569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
Changed lines of the file:
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@@
 			)
 		)
-		(property "Order" "https://www.digikey.com/en/products/detail/maxlinear-inc/SP3485EN-L-TR/2471929"
+		(property "Order" "https://lcsc.com/product-detail/image/SP3485EN-L-TR_C8963.html"
 			(at 232.41 355.6 0)
 			(effects
@@
 			)
 		)
-		(property "Order" "https://www.amazon.ca/FS8205A-TSSOP8-FS8205-CEG8205A-CEG8205/dp/B0BWF4NXFN"
+		(property "Order" "https://icdayroi.com/fs8205a"
 			(at 529.59 49.53 0)
 			(effects
@@
 			)
 		)
-		(property "Order" "https://www.digikey.com/en/products/detail/on-shore-technology-inc/PJ012-8P8C1/6566534"
+		(property "Order" "https://lcsc.com/product-detail/image/R-RJ45S08P-A004_C2902702.html"
 			(at 377.19 173.99 0)
 			(effects
@@
 			)
 		)
-		(property "Order" "https://www.mouser.vn/ProductDetail/Microchip-Technology/MCP1799T-3302H-DB?qs=BJlw7L4Cy7%2F9AvPRs1acXA%3D%3D&srsltid=AfmBOopmPbAsABp1kBvzR_zqpSCa48MAdIcQhqzp9yK27vllvHlsBwub"
+		(property "Order" "https://lcsc.com/product-detail/Voltage-Regulators-Linear-Low-Drop-Out-LDO-Regulators_TECH-PUBLIC-TPMCP1799T-3302H-DB_C42394081.html?s_z=n_MCP1799T-3302H%252FDB"
 			(at 196.85 163.83 0)
 			(effects
@@
 			)
 		)
+		(property "Order" "https://lcsc.com/product-detail/image/DB128V-5-08-2P-GN-S_C2915639.html"
+			(at 304.8 54.61 0)
+			(effects
+				(font
+					(size 1.27 1.27)
+				)
+				(hide yes)
+			)
+		)
 		(pin "2"
 		)
@@
 			)
 		)
+		(property "Order" "https://lcsc.com/product-detail/image/MBR0520_C5204745.html"
+			(at 153.67 86.36 90)
+			(effects
+				(font
+					(size 1.27 1.27)
+				)
+				(hide yes)
+			)
+		)
 		(pin "1"
 		)
@@
 			)
 		)
+		(property "Order" "https://lcsc.com/product-detail/image/DB128V-5-08-2P-GN-S_C2915639.html"
+			(at 306.07 347.98 0)
+			(effects
+				(font
+					(size 1.27 1.27)
+				)
+				(hide yes)
+			)
+		)
 		(pin "2"
 		)
@@
 			)
 		)
+		(property "Order" "https://lcsc.com/product-detail/image/MHK2310RRBTD_C2764897.html"
+			(at 140.97 26.67 0)
+			(effects
+				(font
+					(size 1.27 1.27)
+				)
+				(hide yes)
+			)
+		)
 		(pin "4"
 		)
@@
 			)
 		)
-		(property "Order" "https://www.digikey.com/en/products/detail/maxlinear-inc/SP3485EN-L-TR/2471929"
+		(property "Order" "https://lcsc.com/product-detail/image/SP3485EN-L-TR_C8963.html"
 			(at 220.98 62.23 0)
 			(effects
@@
 			)
 		)
-		(property "Order" "https://linhkienchatluong.vn/ic-nguon/dw01-sot23-6-ic-bao-ve-pin-battery-protection-ic_sp422_ct7133.aspx"
+		(property "Order" "https://lcsc.com/product-detail/image/DW01A_C2927799.html"
 			(at 547.37 38.1 0)
 			(effects
@@
 			)
 		)
-		(property "Order" "https://www.mouser.vn/ProductDetail/CTS-Electronic-Components/445I33D25M00000?qs=FP1Nkeq3mZ9bOUvLGTxcHQ%3D%3D"
+		(property "Order" "https://lcsc.com/product-detail/image/X503225MSB2GI_C112569.html"
 			(at 66.04 257.81 0)
 			(effects
@@
 			)
 		)
-		(property "Order" "https://www.lcsc.com/product-detail/D-Sub-VGA-Connectors_Amphenol-ICC-ID09S33E4GV00LF_C185657.html?s_z=n_db9"
+		(property "Order" "https://lcsc.com/product-detail/D-Sub-VGA-Connectors_XUNPU-D-SUB-DR-9PCM-CB_C19077337.html?s_z=n_db9"
 			(at 35.56 143.51 0)
 			(effects
@@
 			)
 		)
-		(property "Order" "https://www.digikey.com/en/products/detail/microchip-technology/ENC28J60-SS/857584"
+		(property "Order" "https://lcsc.com/product-detail/image/ENC28J60-SS_C8961.html"
 			(at 111.76 247.65 0)
 			(effects
@@
 			)
 		)
-		(property "Order" "https://giadungnhaviet.com/san-pham/pin-sac-cuc-ao-han-chan-ni-mh-3-6v-40mah-3-v40h/"
+		(property "Order" "https://nshopvn.com/product/pin-sac-ni-mh/?variant=144643"
 			(at 502.92 40.64 0)
 			(effects
@@
 			)
 		)
+		(property "Order" "https://lcsc.com/product-detail/image/MHK2310RRBTD_C2764897.html"
+			(at 152.4 320.04 0)
+			(effects
+				(font
+					(size 1.27 1.27)
+				)
+				(hide yes)
+			)
+		)
 		(pin "4"
 		)
@@
 			)
 		)
+		(property "Order" "https://lcsc.com/product-detail/image/CL21A106KOQNNNE_C1713.html"
+			(at 135.89 271.78 0)
+			(effects
+				(font
+					(size 1.27 1.27)
+				)
+				(hide yes)
+			)
+		)
 		(pin "1"
 		)
@@
 			)
 		)
-		(property "Order" "https://www.mouser.vn/ProductDetail/Analog-Devices-Maxim-Integrated/DS3231M%2BTRL?qs=Bakm8ERcljq5PBzSwLfmgg%3D%3D&srsltid=AfmBOorCQu3YM_8BMzXmazTKuCOz4H43YGxirF3dy01P5bAkAlutOfU3"
+		(property "Order" "https://lcsc.com/product-detail/image/DS3231SN-T-R_C9866.html"
 			(at 450.85 60.96 0)
 			(effects
@@
 			(at 237.49 247.65 0)
 			(effects
+				(font
+					(size 1.27 1.27)
+				)
+				(hide yes)
+			)
+		)
+		(property "Order" "https://lcsc.com/product-detail/image/RJ45-334-053-01_C47345453.html"
+			(at 237.49 247.65 0)
+			(effects

Commit message: final link order
Parts:
- D40: Order (none) -> https://lcsc.com/product-detail/image/MBR0520LT1G_C23848.ht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
Changed lines of the file:
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@@
+			)
+		)
+		(property "Order" "https://lcsc.com/product-detail/image/MBR0520LT1G_C23848.html"
+			(at 165.1 379.73 90)
+			(effects
+				(font
+					(size 1.27 1.27)
+				)
+				(hide yes)
 			)
 		)
